File: MA Command Keyboard changed footprint.kicad_pcb (KiCad board)
At the start: 2 copper layers, 195.3 x 216.3 mm, 165 parts, among them SW1 SW_Push, U1 ATmega32U4-A, Y1 16MHz

Commit message: Traces First Draft
Parts:
- moved R2 129.7 mm to (-198.8, 189.5)
- moved R1 129.7 mm to (-200.7, 189.5)
- moved SW1 24.5 mm to (-182.3, 188.1), turned to -90 degrees
- moved R4 19.6 mm to (-202.6, 210.8), turned to 180 degrees
- moved C4 18.5 mm to (-206.6, 206.3), turned to 90 degrees
- moved C1 18.1 mm to (-185.1, 205.2), turned to 180 degrees
- moved C5 17.6 mm to (-193.0, 210.6), turned to 0 degrees
- moved R3 16.7 mm to (-189.1, 189.0), turned to 180 degrees
- moved Y1 16.3 mm to (-185.1, 202.0), turned to 90 degrees
- moved C2 15.5 mm to (-185.1, 198.3), turned to 0 degrees
- moved C7 15.0 mm to (-206.6, 197.5), turned to -90 degrees
- moved C6 13.2 mm to (-189.1, 192.4), turned to 0 degrees
- moved C3 9.63 mm to (-194.8, 191.5), turned to 90 degrees
- moved U1 5.08 mm to (-197.8, 201.7), turned to -90 degrees
Connections:
- MX11 pad 1: cOL1 -> COL1
- MX19 pad 1: cOL1 -> COL1
- MX2 pad 1: cOL1 -> COL1
- MX26 pad 1: cOL1 -> COL1
- MX34 pad 1: cOL1 -> COL1
- MX43 pad 1: cOL1 -> COL1
- MX52 pad 1: cOL1 -> COL1
- MX58 pad 1: cOL1 -> COL1
- MX67 pad 1: cOL1 -> COL1
- U1 pad 10: unconnected-(U1-Pad10) -> ROW1
- U1 pad 11: unconnected-(U1-Pad11) -> ROW2
- U1 pad 22: unconnected-(U1-Pad22) -> COL8
- U1 pad 25: unconnected-(U1-Pad25) -> COL7
- U1 pad 26: unconnected-(U1-Pad26) -> COL6
- U1 pad 27: unconnected-(U1-Pad27) -> COL5
- U1 pad 28: unconnected-(U1-Pad28) -> COL4
- U1 pad 29: unconnected-(U1-Pad29) -> COL3
- U1 pad 30: unconnected-(U1-Pad30) -> COL2
- U1 pad 31: unconnected-(U1-Pad31) -> COL1
- U1 pad 32: unconnected-(U1-Pad32) -> COL0
- U1 pad 36: unconnected-(U1-Pad36) -> ROW8
- U1 pad 37: unconnected-(U1-Pad37) -> ROW7
- U1 pad 38: unconnected-(U1-Pad38) -> ROW6
- U1 pad 39: unconnected-(U1-Pad39) -> ROW5
- U1 pad 40: unconnected-(U1-Pad40) -> ROW4
- U1 pad 41: unconnected-(U1-Pad41) -> ROW3
- U1 pad 9: unconnected-(U1-Pad9) -> ROW0
Routing:
- net COL1: track 0.00 -> 345.0 mm, vias 0 -> 1
- net ROW0: track 214.1 -> 428.7 mm, vias 2 -> 6
- net cOL1: track 211.9 -> 0.00 mm
- net ROW8: track 267.5 -> 461.8 mm, vias 0 -> 2
- net ROW1: track 189.5 -> 377.7 mm, vias 0 -> 6
- net ROW2: track 193.8 -> 362.6 mm, vias 0 -> 6
- net D-: track 7.63 -> 169.5 mm
- net ROW7: track 264.2 -> 426.0 mm, vias 0 -> 2
- net D+: track 7.47 -> 168.9 mm
- net COL0: track 190.5 -> 346.1 mm, vias 0 -> 1
- net GND: track 111.2 -> 260.3 mm, vias 0 -> 4
- net ROW5: track 215.0 -> 354.3 mm, vias 0 -> 4
- net ROW3: track 201.9 -> 339.7 mm, vias 0 -> 4
- net +5V: track 87.4 -> 219.7 mm, vias 6 -> 10
- net ROW6: track 141.9 -> 270.4 mm, vias 0 -> 2
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