File: MA Command Keyboard changed footprint.kicad_sch (KiCad schematic)
At the start: 16 parts, among them SW1 SW_Push, U1 ATmega32U4-A, Y1 16MHz

Commit message: Traces First Draft
Connections:
- net ROW1: now reaches U1.10 (PB2)
- net ROW2: now reaches U1.11 (PB3)
- net ROW8: now reaches U1.36 (PF7)
- net ROW7: now reaches U1.37 (PF6)
- net ROW6: now reaches U1.38 (PF5)
- net ROW5: now reaches U1.39 (PF4)
- net ROW4: now reaches U1.40 (PF1)
- net ROW3: now reaches U1.41 (PF0)
- net ROW0: now reaches U1.9 (PB1)
Changed lines of the file:
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@@
+    )
+  )
+  (global_label "ROW4" (shape input) (at 87.63 101.6 0) (fields_autoplaced)
+    (effects (font (size 1.27 1.27)) (justify left))
+    (property "Intersheet References" "${INTERSHEET_REFS}" (id 0) (at 95.3045 101.5206 0)
+      (effects (font (size 1.27 1.27)) (justify left) hide)
     )
   )
@@
     )
   )
+  (global_label "ROW6" (shape input) (at 87.63 106.68 0) (fields_autoplaced)
+    (effects (font (size 1.27 1.27)) (justify left))
+    (property "Intersheet References" "${INTERSHEET_REFS}" (id 0) (at 95.3045 106.6006 0)
+      (effects (font (size 1.27 1.27)) (justify left) hide)
+    )
+  )
   (global_label "COL6" (shape input) (at 87.63 83.82 0) (fields_autoplaced)
     (effects (font (size 1.27 1.27)) (justify left))
     (property "Intersheet References" "${INTERSHEET_REFS}" (id 0) (at 94.8812 83.7406 0)
+      (effects (font (size 1.27 1.27)) (justify left) hide)
+    )
+  )
+  (global_label "ROW2" (shape input) (at 87.63 45.72 0) (fields_autoplaced)
+    (effects (font (size 1.27 1.27)) (justify left))
+    (property "Intersheet References" "${INTERSHEET_REFS}" (id 0) (at 95.3045 45.6406 0)
       (effects (font (size 1.27 1.27)) (justify left) hide)
     )
@@
     )
   )
+  (global_label "ROW1" (shape input) (at 87.63 43.18 0) (fields_autoplaced)
+    (effects (font (size 1.27 1.27)) (justify left))
+    (property "Intersheet References" "${INTERSHEET_REFS}" (id 0) (at 95.3045 43.1006 0)
+      (effects (font (size 1.27 1.27)) (justify left) hide)
+    )
+  )
+  (global_label "ROW7" (shape input) (at 87.63 109.22 0) (fields_autoplaced)
+    (effects (font (size 1.27 1.27)) (justify left))
+    (property "Intersheet References" "${INTERSHEET_REFS}" (id 0) (at 95.3045 109.1406 0)
+      (effects (font (size 1.27 1.27)) (justify left) hide)
+    )
+  )
   (global_label "D-" (shape input) (at 123.19 39.37 0) (fields_autoplaced)
     (effects (font (size 1.27 1.27)) (justify left))
     (property "Intersheet References" "${INTERSHEET_REFS}" (id 0) (at 128.4455 39.4494 0)
+      (effects (font (size 1.27 1.27)) (justify left) hide)
+    )
+  )
+  (global_label "ROW8" (shape input) (at 87.63 111.76 0) (fields_autoplaced)
+    (effects (font (size 1.27 1.27)) (justify left))
+    (property "Intersheet References" "${INTERSHEET_REFS}" (id 0) (at 95.3045 111.6806 0)
       (effects (font (size 1.27 1.27)) (justify left) hide)
     )
@@
     )
   )
+  (global_label "ROW0" (shape input) (at 87.63 40.64 0) (fields_autoplaced)
+    (effects (font (size 1.27 1.27)) (justify left))
+    (property "Intersheet References" "${INTERSHEET_REFS}" (id 0) (at 95.3045 40.5606 0)
+      (effects (font (size 1.27 1.27)) (justify left) hide)
+    )
+  )
   (global_label "D+" (shape input) (at 31.75 63.5 180) (fields_autoplaced)
     (effects (font (size 1.27 1.27)) (justify right))
@@
     )
   )
+  (global_label "ROW3" (shape input) (at 87.63 99.06 0) (fields_autoplaced)
+    (effects (font (size 1.27 1.27)) (justify left))
+    (property "Intersheet References" "${INTERSHEET_REFS}" (id 0) (at 95.3045 99.1394 0)
+      (effects (font (size 1.27 1.27)) (justify left) hide)
+    )
+  )
   (global_label "COL8" (shape input) (at 87.63 81.28 0) (fields_autoplaced)
     (effects (font (size 1.27 1.27)) (justify left))
@@
       (effects (font (size 1.27 1.27)) (justify left) hide)
     )
+  )
+  (global_label "ROW5" (shape input) (at 87.63 104.14 0) (fields_autoplaced)
+    (effects (font (size 1.27 1.27)) (justify left))
+    (property "Intersheet References" "${INTERSHEET_REFS}" (id 0) (at 95.3045 104.0606 0)
+      (effects (font (size 1.27 1.27)) (justify left) hide)
+    )
